Commit message: add docker

File: src/fetch_description_local/urdf/fetch.urdf (robot description, URDF)
Before this commit: robot fetch, 26 links, 25 joints
Links:
- link base_link: geometry collision mesh filename=package://fetch_description_local/meshes/base_link_collisio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; visual mesh filename=package://fetch_description_local/meshes/base_link.dae
- link bellows_link: geometry collision mesh filename=package://fetch_description_local/meshes/bellows_link_colli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; visual mesh filename=package://fetch_description_local/meshes/bellows_link.STL
- link bellows_link2: geometry collision mesh filename=package://fetch_description_local/meshes/bellows_link_colli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; visual mesh filename=package://fetch_description_local/meshes/bellows_link.STL
- link elbow_flex_link: geometry collision mesh filename=package://fetch_description_local/meshes/elbow_flex_link_co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; visual mesh filename=package://fetch_description_local/meshes/elbow_flex_link.dae
- link estop_link: geometry collision mesh filename=package://fetch_description_local/meshes/estop_link.STL; visual mesh filename=package://fetch_description_local/meshes/estop_link.STL
- link forearm_roll_link: geometry collision mesh filename=package://fetch_description_local/meshes/forearm_roll_link_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; visual mesh filename=package://fetch_description_local/meshes/forearm_roll_link.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
- link gripper_link: geometry collision mesh filename=package://fetch_description_local/meshes/gripper_link.STL; visual mesh filename=package://fetch_description_local/meshes/gripper_link.dae
- link head_pan_link: geometry collision mesh filename=package://fetch_description_local/meshes/head_pan_link_coll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; visual mesh filename=package://fetch_description_local/meshes/head_pan_link.dae
- link head_tilt_link: geometry collision mesh filename=package://fetch_description_local/meshes/head_tilt_link_col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; visual mesh filename=package://fetch_description_local/meshes/head_tilt_link.dae
- link l_gripper_finger_link: geometry collision mesh filename=package://fetch_description_local/meshes/l_gripper_finger_l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; visual mesh filename=package://fetch_description_local/meshes/l_gripper_finger_l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
- link l_wheel_link: geometry collision mesh filename=package://fetch_description_local/meshes/l_wheel_link_colli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; visual mesh filename=package://fetch_description_local/meshes/l_wheel_link.STL
- link laser_link: geometry collision mesh filename=package://fetch_description_local/meshes/laser_link.STL; visual mesh filename=package://fetch_description_local/meshes/laser_link.STL
- link r_gripper_finger_link: geometry collision mesh filename=package://fetch_description_local/meshes/r_gripper_finger_l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; visual mesh filename=package://fetch_description_local/meshes/r_gripper_finger_l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
- link r_wheel_link: geometry collision mesh filename=package://fetch_description_local/meshes/r_wheel_link_colli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; visual mesh filename=package://fetch_description_local/meshes/r_wheel_link.STL
- link shoulder_lift_link: geometry collision mesh filename=package://fetch_description_local/meshes/shoulder_lift_link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; visual mesh filename=package://fetch_description_local/meshes/shoulder_lift_link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
- link shoulder_pan_link: geometry collision mesh filename=package://fetch_description_local/meshes/shoulder_pan_link_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; visual mesh filename=package://fetch_description_local/meshes/shoulder_pan_link.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
- link torso_fixed_link: geometry collision mesh filename=package://fetch_description_local/meshes/torso_fixed_link.S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; visual mesh filename=package://fetch_description_local/meshes/torso_fixed_link.d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
- link torso_lift_link: geometry collision mesh filename=package://fetch_description_local/meshes/torso_lift_link_co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; visual mesh filename=package://fetch_description_local/meshes/torso_lift_link.dae
- link upperarm_roll_link: geometry collision mesh filename=package://fetch_description_local/meshes/upperarm_roll_link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; visual mesh filename=package://fetch_description_local/meshes/upperarm_roll_link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
- link wrist_flex_link: geometry collision mesh filename=package://fetch_description_local/meshes/wrist_flex_link_co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; visual mesh filename=package://fetch_description_local/meshes/wrist_flex_link.dae
- link wrist_roll_link: geometry collision mesh filename=package://fetch_description_local/meshes/wrist_roll_link_co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; visual mesh filename=package://fetch_description_local/meshes/wrist_roll_link.dae
